Commit message: motors_rotating

File: urdf/omni_wheels.urdf.xacro (robot description, xacro)
@@ -33,6 +33,6 @@
     -->
     <gazebo reference="omni_${suffix}_link">
-      <mu1 value="1" />
-      <mu2 value="0.1" />
+      <mu1 value="0.01" />
+      <mu2 value="10" />
       <kp value="10000000.0" />
       <kd value="10000.0" />
@@ -41,19 +41,11 @@
     </gazebo>
     <!-- precisa de parent e origin -->
-    <joint name="omni_${suffix}_joint" type="revolute">
+    <joint name="omni_${suffix}_joint" type="continuous">
       <xacro:insert_block name="joint_pose" />
       <xacro:insert_block name="joint_parent" />
       <child link="omni_${suffix}_link" />
       <axis xyz="0 0 1" rpy="0 0 0" />
-      <limit effort="30" velocity="3.0" lower="${-3.4028235e+38}" upper="${3.4028235e+38}" />
+      <limit effort="30" velocity="3.0" />
     </joint>
-    <gazebo>
-      <plugin
-        filename="gz-sim-joint-controller-system"
-        name="gz::sim::systems::JointController">
-        <joint_name>omni_${suffix}_joint</joint_name>
-        <initial_velocity>0</initial_velocity>
-      </plugin>
-    </gazebo>
   </xacro:macro>
 </robot>

File: urdf/robotino_base.gazebo.xacro (robot description, xacro)
@@ -2,9 +2,5 @@
 <robot xmlns:xacro="http://www.ros.org/wiki/xacro">
     <gazebo>
-        <!-- aqui importamos os plugins que vamos usar -->
-        <plugin
-            filename="gz-sim-joint-state-publisher-system"
-            name="gz::sim::systems::JointStatePublisher">
-        </plugin>
+        <!-- aqui importamos os plugins que vamos usar na simulação -->
         <plugin
             filename="gz-sim-pose-publisher-system"
@@ -20,9 +16,11 @@
             <render_engine>ogre2</render_engine>
         </plugin>
+        <plugin filename="ign_ros2_control-system" name="ign_ros2_control::IgnitionROS2ControlPlugin">
+            <parameters>$(find neo_robotino_sim)/config/motor_velocity_controller.yaml</parameters>
+        </plugin>
     </gazebo>
     <!-- configs do LIDAR -->
     <gazebo reference="lidar_link">
-        <sensor name='gpu_lidar' type='gpu_lidar'>"
-            <topic> lidar </topic>
+        <sensor name='gpu_lidar' type='gpu_lidar'>" <topic> lidar </topic>
             <update_rate> 10 </update_rate>
             <ray>
@@ -47,5 +45,6 @@
                 </range>
             </ray>
-            <always_on>1</always_on>
+            <always_on>
+            1</always_on>
             <visualize>true</visualize>
         </sensor>

File: urdf/robotino_base.urdf.xacro (robot description, xacro)
@@ -86,3 +86,35 @@
         <parent link="structure_link" />
     </xacro:omni_wheel>
+    <ros2_control name="IgnitionSystem" type="system">
+        <hardware>
+            <plugin>ign_ros2_control/IgnitionSystem</plugin>
+        </hardware>
+        <joint name="omni_back_joint">
+            <command_interface name="velocity">
+                <param name="min">-15</param>
+                <param name="max">15</param>
+            </command_interface>
+            <state_interface name="position" />
+            <state_interface name="velocity" />
+            <state_interface name="effort" />
+        </joint>
+        <joint name="omni_left_joint">
+            <command_interface name="velocity">
+                <param name="min">-15</param>
+                <param name="max">15</param>
+            </command_interface>
+            <state_interface name="position" />
+            <state_interface name="velocity" />
+            <state_interface name="effort" />
+        </joint>
+        <joint name="omni_right_joint">
+            <command_interface name="velocity">
+                <param name="min">-15</param>
+                <param name="max">15</param>
+            </command_interface>
+            <state_interface name="position" />
+            <state_interface name="velocity" />
+            <state_interface name="effort" />
+        </joint>
+    </ros2_control>
 </robot>

Commit message: working wheels sim

File: urdf/omni_wheels.urdf.xacro (robot description, xacro)
@@ -33,5 +33,5 @@
     -->
     <gazebo reference="omni_${suffix}_link">
-      <mu1 value="0.01" />
+      <mu1 value="0.2" />
       <mu2 value="10" />
       <kp value="10000000.0" />

File: urdf/robotino_base.urdf.xacro (robot description, xacro)
@@ -79,9 +79,9 @@
     </xacro:omni_wheel>
     <xacro:omni_wheel suffix="left" radius="${wheel_radius}" height="${wheel_height}" mass="0.2">
-        <origin xyz="-0.11631 0.06707 ${(-height/2)+0.01}" rpy="${PI/2} 0 ${PI/3}" />
+        <origin xyz="-0.11631 0.06707 ${(-height/2)+0.01}" rpy="${PI/2} 0 ${PI+PI/3}" />
         <parent link="structure_link" />
     </xacro:omni_wheel>
     <xacro:omni_wheel suffix="right" radius="${wheel_radius}" height="${wheel_height}" mass="0.2">
-        <origin xyz="0.11631 0.06707 ${(-height/2)+0.01}" rpy="${PI/2} 0 ${-PI/3}" />
+        <origin xyz="0.11631 0.06707 ${(-height/2)+0.01}" rpy="${PI/2} 0 ${PI-PI/3}" />
         <parent link="structure_link" />
     </xacro:omni_wheel>

Commit message: add robot meshes

File: urdf/omni_wheels.urdf.xacro (robot description, xacro)
@@ -13,9 +13,6 @@
         <origin xyz="0 0 0" rpy="0 0 0" />
         <geometry>
-          <cylinder radius="${radius}" length="${height}" />
-        </geometry>
-        <material name="white">
-          <color rgba="1 0.8 0.8 1" />
-        </material>
+          <mesh filename="package://neo_robotino_sim/meshes/omni_wheel.dae"/>
+      </geometry>
       </visual>
       <inertial>

File: urdf/robotino_base.urdf.xacro (robot description, xacro)
@@ -23,11 +23,8 @@
         </collision>
         <visual>
-            <origin xyz="0 0 0" rpy="0 0 0" />
+            <origin xyz="0 0 -0.02" rpy="0 0 0" />
             <geometry>
-                <cylinder radius="${radius}" length="${height}" />
+                <mesh filename="package://neo_robotino_sim/meshes/robotino_body.dae"/>
             </geometry>
-            <material name="white">
-                <color rgba="1 0.5 1 1" />
-            </material>
         </visual>
         <inertial>
@@ -72,16 +69,16 @@
         <parent link="structure_link" />
         <child link="lidar_link" />
-        <origin rpy="0 0 0" xyz="-0.1 -0.08 ${(height/2)+0.02}" />
+        <origin rpy="0 0 0" xyz="-0.06 -0.06 ${(height/2)+0.06}" />
     </joint>
     <xacro:omni_wheel suffix="back" radius="${wheel_radius}" height="${wheel_height}" mass="0.2">
-        <origin xyz="-0.13 0 ${(-height/2)+0.01}" rpy="${PI/2} 0 ${PI/2}" />
+        <origin xyz="-0.13 0 ${(-height/2)+(wheel_radius)-0.02}" rpy="${PI/2} 0 ${-PI/2}" />
         <parent link="structure_link" />
     </xacro:omni_wheel>
     <xacro:omni_wheel suffix="right" radius="${wheel_radius}" height="${wheel_height}" mass="0.2">
-        <origin xyz="0.065 -0.11 ${(-height/2)+0.01}" rpy="${PI/2} 0 ${PI+PI/3}" />
+        <origin xyz="0.065 -0.11 ${(-height/2)+(wheel_radius)-0.02}" rpy="${PI/2} 0 ${-PI/3 + PI/2}" />
         <parent link="structure_link" />
     </xacro:omni_wheel>
     <xacro:omni_wheel suffix="left" radius="${wheel_radius}" height="${wheel_height}" mass="0.2">
-        <origin xyz="0.065 0.11 ${(-height/2)+0.01}" rpy="${PI/2} 0 ${-PI/3}" />
+        <origin xyz="0.065 0.11 ${(-height/2)+(wheel_radius)-0.02}" rpy="${PI/2} 0 ${PI/3 + PI/2}" />
         <parent link="structure_link" />
     </xacro:omni_wheel>

Commit message: started implementing odom

File: urdf/omni_wheels.urdf.xacro (robot description, xacro)
@@ -11,5 +11,5 @@
       </collision>
       <visual>
-        <origin xyz="0 0 0" rpy="0 0 0" />
+        <origin xyz="0 0 0.005" rpy="0 0 0" />
         <geometry>
           <mesh filename="package://neo_robotino_sim/meshes/omni_wheel.dae"/>
@@ -43,5 +43,5 @@
       <child link="omni_${suffix}_link" />
       <axis xyz="0 0 1" rpy="0 0 0" />
-      <limit effort="30" velocity="3.0" />
+      <limit effort="30" velocity="25.0" />
     </joint>
   </xacro:macro>
