Commit message: fix LiDAR and add rviz config

File: urdf/robotino_base.gazebo.xacro (robot description, xacro)
@@ -22,7 +22,19 @@
     <!-- configs do LIDAR -->
     <gazebo reference="lidar_link">
-        <sensor name='gpu_lidar' type='gpu_lidar'>" <topic> lidar </topic>
+        <sensor name='gpu_lidar' type='gpu_lidar'>
+            <topic> /lidar </topic>
+            <!--
+                solução para mudar o frame_id da mensagem
+                https://github.com/gazebosim/gz-sensors/pull/195
+                porém não funciona nesa versão do gazebo
+            -->
+            <frame_id>lidar_link</frame_id>
+            <!--
+                essa issue fala mais sobre isso e da a solução
+                https://github.com/gazebosim/gz-sensors/issues/384
+            -->
+            <ignition_frame_id>lidar_link</ignition_frame_id>
             <update_rate> 10 </update_rate>
-            <ray>
+            <lidar>
                 <scan>
                     <horizontal>
@@ -44,8 +56,11 @@
                     <resolution>0.01</resolution>
                 </range>
-            </ray>
-            <always_on>
-            1</always_on>
-            <visualize>true</visualize>
+                <noise>
+                    <type>gaussian</type>
+                    <mean>0</mean>
+                    <stddev>0.01</stddev>
+                </noise>
+            </lidar>
+            <always_on>1</always_on>
         </sensor>
     </gazebo>

File: urdf/robotino_base.urdf.xacro (robot description, xacro)
@@ -72,16 +72,16 @@
         <parent link="structure_link" />
         <child link="lidar_link" />
-        <origin rpy="0 0 0" xyz="0.1 0.1 ${(height/2)+0.02}" />
+        <origin rpy="0 0 0" xyz="-0.1 -0.08 ${(height/2)+0.02}" />
     </joint>
     <xacro:omni_wheel suffix="back" radius="${wheel_radius}" height="${wheel_height}" mass="0.2">
-        <origin xyz="0 -0.13426 ${(-height/2)+0.01}" rpy="${PI/2} 0 0" />
+        <origin xyz="-0.13 0 ${(-height/2)+0.01}" rpy="${PI/2} 0 ${PI/2}" />
+        <parent link="structure_link" />
+    </xacro:omni_wheel>
+    <xacro:omni_wheel suffix="right" radius="${wheel_radius}" height="${wheel_height}" mass="0.2">
+        <origin xyz="0.065 -0.11 ${(-height/2)+0.01}" rpy="${PI/2} 0 ${PI+PI/3}" />
         <parent link="structure_link" />
     </xacro:omni_wheel>
     <xacro:omni_wheel suffix="left" radius="${wheel_radius}" height="${wheel_height}" mass="0.2">
-        <origin xyz="-0.11631 0.06707 ${(-height/2)+0.01}" rpy="${PI/2} 0 ${PI+PI/3}" />
-        <parent link="structure_link" />
-    </xacro:omni_wheel>
-    <xacro:omni_wheel suffix="right" radius="${wheel_radius}" height="${wheel_height}" mass="0.2">
-        <origin xyz="0.11631 0.06707 ${(-height/2)+0.01}" rpy="${PI/2} 0 ${PI-PI/3}" />
+        <origin xyz="0.065 0.11 ${(-height/2)+0.01}" rpy="${PI/2} 0 ${-PI/3}" />
         <parent link="structure_link" />
     </xacro:omni_wheel>

Commit message: Fixed navigation guidance and added distance sensors to the gazebo

File: urdf/robotino_base.gazebo.xacro (robot description, xacro)
@@ -65,3 +65,50 @@
         </sensor>
     </gazebo>
+    <xacro:macro name="add_sensor_plugins" params="suffix">
+        <gazebo reference="dist_sensor_${suffix}_link">
+            <sensor name='distance_sensor_${suffix}' type='gpu_lidar'>
+                <topic>/dist_sensor_${suffix} </topic>
+                <frame_id>dist_sensor_${suffix}_link</frame_id>
+                <ignition_frame_id>dist_sensor_${suffix}_link</ignition_frame_id>
+                <update_rate>10</update_rate>
+                <lidar>
+                    <scan>
+                        <horizontal>
+                            <samples>10</samples>
+                            <resolution>1</resolution>
+                            <min_angle>-0.05</min_angle>
+                            <max_angle>0.05</max_angle>
+                        </horizontal>
+                        <vertical>
+                            <samples>1</samples>
+                            <resolution>0.01</resolution>
+                            <min_angle>0</min_angle>
+                            <max_angle>0</max_angle>
+                        </vertical>
+                    </scan>
+                    <range>
+                        <min>0.04</min>
+                        <max>0.01</max>
+                        <resolution>0.01</resolution>
+                    </range>
+                    <noise>
+                        <type>gaussian</type>
+                        <mean>0</mean>
+                        <stddev>0.01</stddev>
+                    </noise>
+                </lidar>
+                <always_on>1</always_on>
+            </sensor>
+        </gazebo>
+    </xacro:macro>
+    <!-- chama macro para criar os plugins -->
+    <xacro:add_sensor_plugins suffix="0"/>
+    <xacro:add_sensor_plugins suffix="1"/>
+    <xacro:add_sensor_plugins suffix="2"/>
+    <xacro:add_sensor_plugins suffix="3"/>
+    <xacro:add_sensor_plugins suffix="4"/>
+    <xacro:add_sensor_plugins suffix="5"/>
+    <xacro:add_sensor_plugins suffix="6"/>
+    <xacro:add_sensor_plugins suffix="7"/>
+    <xacro:add_sensor_plugins suffix="8"/>
 </robot>

File: urdf/robotino_base.urdf.xacro (robot description, xacro)
@@ -4,4 +4,5 @@
     <xacro:include filename="omni_wheels.urdf.xacro" />
     <xacro:include filename="robotino_base.gazebo.xacro" />
+    <xacro:include filename="dist_sensor.urdf.xacro" />
     <!-- Constants for robot dimensions -->
     <xacro:property name="PI" value="3.1415926535897931" />
@@ -68,9 +69,10 @@
         <parent link="base_link" />
         <child link="base_footprint" />
-        <origin xyz="0 0 ${(-height/2)+(-wheel_radius)+(wheel_clearance)}" rpy="0 0 0" />
+        <origin xyz="0 0 ${((-height/2)+(-wheel_radius)+(wheel_clearance))}" rpy="0 0 ${PI}" />
     </joint>
     <joint name="base_to_structure" type="fixed">
         <parent link="base_link" />
         <child link="structure_link" />
+        <origin xyz="0 0 0" rpy="0 0 ${PI}" />
     </joint>
     <joint name="structure_to_lidar" type="fixed">
@@ -91,4 +93,31 @@
         <parent link="structure_link" />
     </xacro:omni_wheel>
+    <xacro:dist_sensor suffix="0" mass="0.0035" robot_radius="${radius}">
+        <parent link="structure_link" />
+    </xacro:dist_sensor>
+    <xacro:dist_sensor suffix="1" mass="0.0035" robot_radius="${radius}">
+        <parent link="structure_link" />
+    </xacro:dist_sensor>
+    <xacro:dist_sensor suffix="2" mass="0.0035" robot_radius="${radius}">
+        <parent link="structure_link" />
+    </xacro:dist_sensor>
+    <xacro:dist_sensor suffix="3" mass="0.0035" robot_radius="${radius}">
+        <parent link="structure_link" />
+    </xacro:dist_sensor>
+    <xacro:dist_sensor suffix="4" mass="0.0035" robot_radius="${radius}">
+        <parent link="structure_link" />
+    </xacro:dist_sensor>
+    <xacro:dist_sensor suffix="5" mass="0.0035" robot_radius="${radius}">
+        <parent link="structure_link" />
+    </xacro:dist_sensor>
+    <xacro:dist_sensor suffix="6" mass="0.0035" robot_radius="${radius}">
+        <parent link="structure_link" />
+    </xacro:dist_sensor>
+    <xacro:dist_sensor suffix="7" mass="0.0035" robot_radius="${radius}">
+        <parent link="structure_link" />
+    </xacro:dist_sensor>
+    <xacro:dist_sensor suffix="8" mass="0.0035" robot_radius="${radius}">
+        <parent link="structure_link" />
+    </xacro:dist_sensor>
     <ros2_control name="IgnitionSystem" type="system">
         <hardware>
